Commit message: addded ros2_control but does not work

File: description/lidar.xacro (robot description, xacro)
@@ -44,5 +44,5 @@
             <plugin name='laser_controller' filename='libgazebo_ros_ray_sensor.so'>
                 <ros>
-                    <argument>--ros-args --remap ~/out:=scan</argument>  <!--the one said in video is deprecated-->
+                    <argument>~/out:=scan</argument>  <!--the one said in video is deprecated-->
                 </ros>
                 <output_type>sensor_msgs/LaserScan</output_type>

File: description/robot.urdf.xacro (robot description, xacro)
@@ -4,3 +4,4 @@
     <xacro:include filename="lidar.xacro"/>
     <xacro:include filename='gazebo_control.xacro'/>
+     <!-- <xacro:include filename='ros2_control.xacro'/> -->
 </robot>

File: description/robot_core.xacro (robot description, xacro)
@@ -19,4 +19,12 @@
     <!-- BASE LINK -->
     <link name="base_link">
+    </link>
+    <!-- BASE FOOTPRINT -->
+    <joint name="base_footprint_joint" type="fixed">
+        <parent link="base_link" />
+        <child link="base_footprint" />
+        <origin xyz="0 0 0" rpy="0 0 0" />
+    </joint>
+    <link name='base_footprint'>
     </link>
     <!-- CHASSIS LINK -->
