Commit message: LiDAR added with a custom world

File: description/gazebo_control.xacro (robot description, xacro)
@@ -7,4 +7,5 @@
              <right_joint>right_wheel_joint</right_joint>
              <wheel_separation>0.35</wheel_separation>
+             <wheel_diameter>0.1</wheel_diameter>
              <!-- Limits -->
              <max_wheel_torque>200.0</max_wheel_torque>

File: description/robot.urdf.xacro (robot description, xacro)
@@ -1,5 +1,6 @@
 <?xml version="1.0"?>
 <robot xmlns:xacro="http://www.ros.org/wiki/xacro"  name="robot">
-    <xacro:include filename="robot_core.xacro" />
+    <xacro:include filename="robot_core.xacro"/>
+    <xacro:include filename="lidar.xacro"/>
     <xacro:include filename='gazebo_control.xacro'/>
 </robot>

File: description/robot_core.xacro (robot description, xacro)
@@ -13,4 +13,7 @@
     <material name="black">
         <color rgba="0 0 0 1"/>
+    </material>
+    <material name="red">
+        <color rgba="1 0 0 1"/>
     </material>
     <!-- BASE LINK -->

Commit message: ros2_control works

File: description/gazebo_control.xacro (robot description, xacro)
@@ -4,17 +4,17 @@
         <plugin name="diff_drive" filename="libgazebo_ros_diff_drive.so">
             <!-- Wheel Info -->
-             <left_joint>left_wheel_joint</left_joint>
-             <right_joint>right_wheel_joint</right_joint>
-             <wheel_separation>0.35</wheel_separation>
-             <wheel_diameter>0.1</wheel_diameter>
-             <!-- Limits -->
-             <max_wheel_torque>200.0</max_wheel_torque>
-             <max_wheel_accelaration>10.0</max_wheel_accelaration>
-             <!-- Output -->
-                <odometry_frame>odom</odometry_frame>
-                <robot_base_frame>base_link</robot_base_frame>
-                <publish_odom>true</publish_odom>
-                <publish_odom_tf>true</publish_odom_tf>
-                <publish_wheel_tf>true</publish_wheel_tf>
+            <left_joint>left_wheel_joint</left_joint>
+            <right_joint>right_wheel_joint</right_joint>
+            <wheel_separation>0.35</wheel_separation>
+            <wheel_diameter>0.1</wheel_diameter>
+            <!-- Limits -->
+            <max_wheel_torque>200.0</max_wheel_torque>
+            <max_wheel_accelaration>10.0</max_wheel_accelaration>
+            <!-- Output -->
+            <odometry_frame>odom</odometry_frame>
+            <robot_base_frame>base_link</robot_base_frame>
+            <publish_odom>true</publish_odom>
+            <publish_odom_tf>true</publish_odom_tf>
+            <publish_wheel_tf>true</publish_wheel_tf>
         </plugin>
     </gazebo>

File: description/lidar.xacro (robot description, xacro)
@@ -44,4 +44,6 @@
             <plugin name='laser_controller' filename='libgazebo_ros_ray_sensor.so'>
                 <ros>
+                    <argument>--ros-args</argument>
+                    <argument>--remap</argument>
                     <argument>~/out:=scan</argument>  <!--the one said in video is deprecated-->
                 </ros>

File: description/robot.urdf.xacro (robot description, xacro)
@@ -3,5 +3,5 @@
     <xacro:include filename="robot_core.xacro"/>
     <xacro:include filename="lidar.xacro"/>
-    <xacro:include filename='gazebo_control.xacro'/>
-     <!-- <xacro:include filename='ros2_control.xacro'/> -->
+    <!-- <xacro:include filename='gazebo_control.xacro'/> -->
+    <xacro:include filename="ros2_control.xacro"/>
 </robot>

File: description/robot_core.xacro (robot description, xacro)
@@ -26,5 +26,5 @@
         <origin xyz="0 0 0" rpy="0 0 0" />
     </joint>
-    <link name='base_footprint'>
+    <link name="base_footprint">
     </link>
     <!-- CHASSIS LINK -->
@@ -52,5 +52,5 @@
         </xacro:inertial_box>
     </link>
-    <gazebo reference='chassis'>
+    <gazebo reference="chassis">
         <material>Gazebo/white</material>
     </gazebo>
@@ -78,5 +78,5 @@
         </xacro:inertial_cylinder>
     </link>
-    <gazebo reference='left_wheel'>
+    <gazebo reference="left_wheel">
         <material>Gazebo/Blue</material>
     </gazebo>
@@ -104,5 +104,5 @@
         </xacro:inertial_cylinder>
     </link>
-    <gazebo reference='right_wheel'>
+    <gazebo reference="right_wheel">
         <material>Gazebo/Blue</material>
     </gazebo>
@@ -129,5 +129,5 @@
         </xacro:inertial_sphere>
     </link>
-    <gazebo reference='castor_wheel'>
+    <gazebo reference="castor_wheel">
         <material>Gazebo/Black</material>
         <mu1 value="0.001"/>

File: description/ros2_control.xacro (robot description, xacro)
@@ -1,29 +1,30 @@
 <?xml version="1.0"?>
 <robot xmlns:xacro="http://www.ros.org/wiki/xacro">
-    <ros2_control name='GazeboControl' type='system'>
+    <ros2_control name="GazeboSystem" type="system">
         <hardware>
             <plugin>gazebo_ros2_control/GazeboSystem</plugin>
         </hardware>
-        <joint name='left_wheel_joint'>
-            <command_interface name='velocity'>
-                <param name='min'>-10</param>
-                <param name='max'>10</param>
+        <joint name="left_wheel_joint">
+            <command_interface name="velocity">
+                <param name="min">-10</param>
+                <param name="max">10</param>
             </command_interface>
-            <state_interface name='velocity'/>
-            <state_interface name='position'/>
+            <state_interface name="velocity"/>
+            <state_interface name="position"/>
         </joint>
-        <joint name='right_wheel_joint'>
-            <command_interface name='velocity'>
-                <param name='min'>-10</param>
-                <param name='max'>10</param>
+        <joint name="right_wheel_joint">
+            <command_interface name="velocity">
+                <param name="min">-10</param>
+                <param name="max">10</param>
             </command_interface>
-            <state_interface name='velocity'/>
-            <state_interface name='position'/>
+            <state_interface name="velocity"/>
+            <state_interface name="position"/>
         </joint>
     </ros2_control>
-    <gazdebo>
-        <plugin name='gazebo_ros2_control' filename='libgazebo_ros2_control.so'>
-            <parameters>$(find my_bot)/config/controllers.yaml</parameters>
+    <gazebo>
+        <plugin name="gazebo_ros2_control" filename="libgazebo_ros2_control.so">
+            <parameters>/home/subham/projects/my_robot/src/my_bot/config/controllers.yaml</parameters>
+            <!-- <parameters>$(find my_bot)/config/controller_manager.yaml</parameters> -->
         </plugin>
-    </gazdebo>
+    </gazebo>
 </robot>
